Commit message: add yaml file

File: turtle_brick/urdf/robot.urdf.xacro (robot description, xacro)
@@ -1,5 +1,6 @@
 <robot name="myfirst" xmlns:xacro="http://wiki.ros.org/wiki/xacro">
+<xacro:property name="prop" value="${xacro.load_yaml('$(find turtle_brick)/turtle.yaml')['/**']['ros__parameters']}"/>
 <xacro:property name="base_length" value="2"/>
-<xacro:property name="base_width" value="2"/>
+<xacro:property name="base_width" value="${prop['base_width']}"/>
 <xacro:property name="base_height" value="2"/>
 <xacro:property name="plat_radius" value="2"/>
@@ -8,5 +9,5 @@
 <xacro:property name="stem_length" value="1"/>
 <xacro:property name="wheel_thickness" value="0.3"/>
-<xacro:property name="wheel_radius" value="0.5"/>
+<xacro:property name="wheel_radius" value="${prop['wheel_radius']}"/>
   <!--base link & cyl-link-->
   <link name="base_link">
